File: audio-mixer.kicad_pcb (KiCad board)
At the start: 2 copper layers, 66 parts, among them J1 Power Input, J2 Stereo Input 1, J3 Stereo Input 2, J4 Stereo Input 3, J5 Stereo Input 4, J6 Conn_01x05, J7 Headphones Output, J8 Speaker Output, U1 TL072, U2 LD1117S50TR_SOT223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

Commit message: General board organization
Parts:
- moved J7 156.0 mm to (259.1, 38.1), turned to 180 degrees
- moved J8 120.2 mm to (259.1, 49.5), turned to 180 degrees
- moved R2 114.6 mm to (236.7, 49.5)
- moved R1 111.5 mm to (237.5, 47.0)
- moved TP20 104.0 mm to (227.1, 82.0)
- moved TP12 104.0 mm to (233.8, 83.1)
- moved TP14 104.0 mm to (230.4, 83.1)
- moved TP11 104.0 mm to (223.1, 84.5)
- moved TP15 104.0 mm to (226.4, 85.0)
- moved U1 97.2 mm to (238.8, 39.4)
- moved TP22 95.8 mm to (222.8, 65.2)
- moved TP21 95.8 mm to (226.2, 65.2)
- moved TP24 95.8 mm to (216.1, 65.2)
- moved TP23 95.8 mm to (219.4, 65.2)
- moved TP13 94.2 mm to (232.4, 78.7)
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Routing:
- net /Attenuation/RIGHT_1: track 0.00 -> 1.52 mm
- net /Attenuation/LEFT_1: track 0.00 -> 1.52 mm
- added copper zone on B.Cu, net GND

Commit message: Input layout
Parts:
- moved TP13 124.9 mm to (109.3, 57.3)
- moved TP14 122.4 mm to (109.3, 65.4)
- moved TP8 121.8 mm to (109.3, 83.9)
- moved TP7 118.3 mm to (109.3, 75.8)
- moved TP16 118.2 mm to (109.3, 81.7)
- moved TP15 117.6 mm to (109.3, 73.5)
- moved TP5 116.6 mm to (109.3, 59.6)
- moved TP12 114.4 mm to (119.4, 85.1)
- moved TP6 112.1 mm to (109.3, 67.7)
- moved TP9 110.1 mm to (119.4, 60.3)
- moved TP17 106.9 mm to (119.4, 57.8)
- moved TP10 105.7 mm to (119.4, 68.6)
- moved TP11 104.1 mm to (119.4, 74.9)
- moved TP18 102.8 mm to (119.4, 65.4)
- moved TP19 81.6 mm to (149.2, 81.9)
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Connections:
- U4 pad 14: Net-(U4-Pad14) -> (no net)
- U5 pad 14: Net-(U5-Pad14) -> (no net)
- U6 pad 12: Net-(TP18-Pad1) -> Net-(TP17-Pad1)
- U6 pad 13: Net-(R16-Pad2) -> Net-(R15-Pad2)
- U6 pad 14: Net-(R16-Pad2) -> Net-(R15-Pad2)
- U6 pad 5: Net-(TP17-Pad1) -> Net-(TP18-Pad1)
- U6 pad 6: Net-(R15-Pad2) -> Net-(R16-Pad2)
- U6 pad 7: Net-(R15-Pad2) -> Net-(R16-Pad2)
Routing:
- net GND: track 0.00 -> 40.6 mm
- net Net-(TP17-Pad1): track 0.00 -> 15.7 mm
- net Net-(TP10-Pad1): track 0.00 -> 15.7 mm
- net +5V: track 0.00 -> 13.8 mm
- net Net-(C6-Pad1): track 0.00 -> 11.8 mm
- net Net-(C3-Pad1): track 0.00 -> 11.8 mm
- net Net-(C1-Pad1): track 0.00 -> 11.8 mm
- net Net-(C8-Pad1): track 0.00 -> 11.8 mm
- net Net-(R7-Pad2): track 0.00 -> 8.03 mm, vias 0 -> 1
- net Net-(R16-Pad2): track 0.00 -> 8.03 mm, vias 0 -> 1
- net Net-(TP19-Pad1): track 0.00 -> 6.86 mm
- net Net-(TP12-Pad1): track 0.00 -> 6.81 mm
- net Net-(TP18-Pad1): track 0.00 -> 6.78 mm
- net Net-(TP9-Pad1): track 0.00 -> 6.64 mm
- net +2V5: track 0.00 -> 6.30 mm
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
Commit message: Complete PCB layout rev. v01
Parts:
- added #LOGO2: OSHW-Logo_5.7x6mm_SilkScreen, Symbol:OSHW-Logo_5.7x6mm_SilkScreen, B.Cu at (116.2, 70.5)
- added H1: MountingHole, MountingHole:MountingHole_3.7mm, F.Cu at (129.2, 51.1)
- added H2: MountingHole, MountingHole:MountingHole_3.7mm, F.Cu at (129.2, 90.2)
- added H3: MountingHole, MountingHole:MountingHole_3.7mm, F.Cu at (151.6, 51.1)
- added J9: Conn_01x05, Connector_PinHeader_2.54mm:PinHeader_1x05_P2.54mm_Horizontal, F.Cu at (110.0, 54.5)
- moved U1 105.3 mm to (138.2, 70.6), turned to 270 degrees
- moved TP1 102.3 mm to (134.2, 69.5)
- moved J7 101.4 mm to (161.4, 65.5)
- moved J8 101.4 mm to (161.4, 77.0)
- moved R2 101.2 mm to (138.8, 75.2), turned to 180 degrees
- moved R1 100.5 mm to (138.8, 66.0), turned to 180 degrees
- moved TP2 100.2 mm to (134.2, 71.8)
- moved TP4 92.6 mm to (142.1, 71.8), turned to 180 degrees
- moved TP3 88.8 mm to (142.1, 69.5), turned to 180 degrees
- moved TP21 79.7 mm to (149.2, 86.0), turned to 270 degrees
- moved TP23 76.7 mm to (143.3, 56.5)
- moved TP22 75.8 mm to (149.2, 83.4), turned to 270 degrees
- moved TP24 75.3 mm to (143.3, 84.5)
- moved J6 50.6 mm to (120.1, 86.8), turned to 270 degrees
- moved U7 42.0 mm to (124.8, 78.7)
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Connections:
- J6 pad 1: /Attenuation/SCL -> /Attenuation/SDA
- J6 pad 2: /Attenuation/SDA -> /Attenuation/SCL
- J6 pad 3: /Attenuation/A0 -> /Attenuation/A0_2
- J6 pad 4: /Attenuation/A1 -> /Attenuation/A1_2
- J6 pad 5: /Attenuation/~RESET -> /Attenuation/~RESET_2
- R15 pad 1: Net-(R15-Pad1) -> /Attenuation/RIGHT_COMBINED
- R16 pad 1: Net-(R15-Pad1) -> /Attenuation/RIGHT_COMBINED
- R17 pad 1: Net-(R15-Pad1) -> /Attenuation/RIGHT_COMBINED
- R18 pad 1: Net-(R15-Pad1) -> /Attenuation/RIGHT_COMBINED
- U4 pad 15: /Attenuation/~RESET -> /Attenuation/~RESET_1
- U4 pad 16: /Attenuation/A1 -> /Attenuation/A1_1
- U4 pad 4: /Attenuation/A0 -> /Attenuation/A0_1
- U5 pad 15: /Attenuation/~RESET -> /Attenuation/~RESET_2
- U5 pad 16: /Attenuation/A1 -> /Attenuation/A1_2
- U5 pad 4: /Attenuation/A0 -> /Attenuation/A0_2
- U7 pad 12: Net-(TP20-Pad1) -> Net-(TP19-Pad1)
- U7 pad 13: Net-(R18-Pad2) -> Net-(R17-Pad2)
- U7 pad 14: Net-(R18-Pad2) -> Net-(R17-Pad2)
- U7 pad 5: Net-(TP19-Pad1) -> Net-(TP20-Pad1)
- U7 pad 6: Net-(R17-Pad2) -> Net-(R18-Pad2)
- U7 pad 7: Net-(R17-Pad2) -> Net-(R18-Pad2)
Routing:
- net /Attenuation/SCL: track 0.00 -> 112.2 mm, vias 0 -> 2
- net +12V: track 0.00 -> 110.2 mm, vias 0 -> 4
- net /Attenuation/SDA: track 0.00 -> 104.1 mm, vias 0 -> 2
- net +2V5: track 6.30 -> 102.7 mm, vias 0 -> 10
- net +5V: track 13.8 -> 83.6 mm, vias 0 -> 7
- net GND: track 40.6 -> 81.6 mm, vias 0 -> 6
- net /Attenuation/LEFT_COMBINED: track 0.00 -> 37.7 mm, vias 0 -> 1
- net /Attenuation/RIGHT_COMBINED: track 0.00 -> 34.9 mm
- net /LEFT_OUT: track 0.00 -> 21.3 mm
- net /Attenuation/~RESET_1: track 0.00 -> 18.6 mm, vias 0 -> 1
- net Net-(J7-PadRN): track 0.00 -> 17.7 mm
- net Net-(J7-PadTN): track 0.00 -> 16.0 mm
- net /Attenuation/A1_1: track 0.00 -> 16.0 mm, vias 0 -> 1
- net /RIGHT_OUT: track 0.00 -> 15.4 mm
- net /Attenuation/~RESET_2: track 0.00 -> 12.7 mm, vias 0 -> 1
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Other:
- board outline added: 66 x 39.1 mm
- board text added: "Audio Mixer"
- board text added: "Benjamin Ward"
- board text added: "Headphones"
- board text added: "Input 1"
- board text added: "Input 2"
- board text added: "Input 3"
- board text added: "Input 4"
- board text added: "Inputs"
- board text added: "Output 1 (Headphones)"
- board text added: "Output 2 (Speaker)"
- board text added: "QMix"
- board text added: "Rev. v01"
- board text added: "Speaker"
